Commit message: mapping succeed

File: src/slam_tutorials/urdf/first_model.urdf (robot description, URDF)
Before this commit: robot myfirst, 3 links, 2 joints
Links:
- added link laser; visual cylinder length=0.04 radius=0.038
- link left_wheel: geometry visual cylinder length=0.03 radius=0.055
- link right_wheel: geometry visual cylinder length=0.03 radius=0.055
Joints:
- added joint base_to_laser: type fixed, parent base_link, child laser, origin xyz=0 0 0.055
- joint base_to_left_wheel: origin (none) -> xyz=0 -0.22 0
- joint base_to_right_wheel: origin (none) -> xyz=0 0.22 0
